Commit message: Squashed 'euroc_stage_2_simulation/' changes from 54aba7e..5086fe4
5086fe4 Merge pull request #12 from ethz-asl/fix/drag_constant
d96e0c1 fixed motor drag constant

git-subtree-dir: euroc_stage_2_simulation
git-subtree-split: 5086fe46cdc4ecae6ece4d4b1b74809a114c44c7

File: euroc_hex_description/urdf/euroc_hex.xacro (robot description, xacro)
@@ -42,5 +42,5 @@
   <xacro:property name="back_propeller_x" value="-0.21561" />
   <xacro:property name="back_propeller_y" value="0.12535" />
-  <xacro:property name="rotor_drag_coefficient" value="0.038" />
+  <xacro:property name="rotor_drag_coefficient" value="2.0673e-04" />
   <xacro:property name="rolling_moment_coefficient" value="0.0" />
   <!-- Property Blocks -->
