Commit message: dodan rotors simulator

File: euroc_stage_2_simulation/euroc_hex_description/urdf/euroc_hex.xacro (robot description, xacro)
@@ -18,5 +18,5 @@
 <robot name="euroc_hex" xmlns:xacro="http://ros.org/wiki/xacro">
   <!-- Properties -->
-  <xacro:property name="namespace" value="$(arg mav_name)" />
+  <xacro:property name="namespace" value="$(arg namespace)" />
   <xacro:property name="rotor_velocity_slowdown_sim" value="10" />
   <xacro:property name="use_mesh_file" value="true" />

Commit message: 23.6 verzija

File: euroc_stage_2_simulation/euroc_hex_description/urdf/euroc_hex.xacro (robot description, xacro)
@@ -18,5 +18,5 @@
 <robot name="euroc_hex" xmlns:xacro="http://ros.org/wiki/xacro">
   <!-- Properties -->
-  <xacro:property name="namespace" value="$(arg namespace)" />
+  <xacro:property name="namespace" value="$(arg mav_name)" />
   <xacro:property name="rotor_velocity_slowdown_sim" value="10" />
   <xacro:property name="use_mesh_file" value="true" />
